File: tp/tp.sch (KiCad schematic (older format))
At the start: 22 parts, among them J1 Conn_01x02, J2 Conn_01x04, T1 ZMPT101B, U1 LM358

Commit message: Agregado de: footprints, descripcion y fabricante
Parts:
- C1, C2, C3, C4, C5: footprint (none) -> Capacitor_SMD:C_0805_2012Metric
- D1: footprint (none) -> LED_SMD:LED_1206_3216Metric
- J1: footprint (none) -> TerminalBlock_Phoenix:TerminalBlock_Phoenix_MKDS-1,5-2-5.08_1x02_P5.08mm_Horizontal; Desc (none) -> PCB terminal block - MKDSN 2,5/ 2-5,08; Digikey# (none) -> 277-5893-ND; Manf (none) -> Phoenix Contact; Manf# (none) -> 1888687
- J2: footprint (none) -> Connector_PinHeader_2.54mm:PinHeader_1x04_P2.54mm_Vertical
- R1, R10, R11, R2, R3, R4, R5, R6, R7, R8, R9: footprint (none) -> Resistor_SMD:R_1206_3216Metric
- RV1: value R_POT -> 100K; footprint (none) -> Resistor_SMD:R_1206_3216Metric; Desc (none) -> TRIMMER 100K OHM 0.5W PC PIN TOP; Digikey#  (none) -> 3296W-104LF-ND; Manf (none) -> Bourns Inc.; Manf# (none) -> 3296W-1-104LF
- T1: footprint XFMR_ZMPT101B -> ZMPT101B:XFMR_ZMPT101B; Desc (none) -> Current-type Voltage Transformer; Digikey# (none) -> N/A; Manf (none) -> Qingxian Zeming Langxi Electronic; Manf# (none) -> ZMPT101B
- U1: footprint (none) -> Package_SO:SOP-8_3.9x4.9mm_P1.27mm; Desc (none) -> LM358, Dual Operational Amplifiers; Digikey#  (none) -> LM358AMXTR-ND; Manf (none) -> Texas Instruments; Manf# (none) -> LM358AMX
- U1: footprint (none) -> Package_SO:SOP-8_3.9x4.9mm_P1.27mm
Other:
- note added: "Gain Adjustment"
Changed lines of the file:
@@
 Rev "1"
 Comp ""
-Comment1 "Revisor: "
-Comment2 "Autor: Cristian Trinidad"
-Comment3 ""
+Comment1 "Creative Commons Attribution-NonCommercial-ShareAlike 4.0 International License"
+Comment2 "Revisor: Felipe Calcavecchia"
+Comment3 "Autor: Cristian Trinidad"
 Comment4 ""
 $EndDescr
@@
 F 0 "T1" H 2666 3840 50  0000 C CNN
 F 1 "ZMPT101B" H 2666 3749 50  0000 C CNN
-F 2 "XFMR_ZMPT101B" H 2600 3450 50  0001 L BNN
-F 3 "" H 2600 3450 50  0001 L BNN
+F 2 "ZMPT101B:XFMR_ZMPT101B" H 2600 3450 50  0001 L BNN
+F 3 "https://www.datasheet4u.com/datasheet-pdf/ZemingLangxi/ZMPT101B/pdf.php?id=1381510" H 2600 3450 50  0001 L BNN
+F 4 "Qingxian Zeming Langxi Electronic" H 2600 3450 50  0001 C CNN "Manf"
+F 5 "ZMPT101B" H 2600 3450 50  0001 C CNN "Manf#"
+F 6 "Current-type Voltage Transformer" H 2600 3450 50  0001 C CNN "Desc"
+F 7 "N/A" H 2600 3450 50  0001 C CNN "Digikey#"
 	1    2600 3450
 	1    0    0    -1
@@
 F 0 "R1" V 1693 3250 50  0000 C CNN
 F 1 "820K" V 1784 3250 50  0000 C CNN
-F 2 "" V 1830 3250 50  0001 C CNN
+F 2 "Resistor_SMD:R_1206_3216Metric" V 1830 3250 50  0001 C CNN
 F 3 "~" H 1900 3250 50  0001 C CNN
 	1    1900 3250
@@
 F 0 "R3" H 3570 3496 50  0000 L CNN
 F 1 "100" H 3570 3405 50  0000 L CNN
-F 2 "" V 3430 3450 50  0001 C CNN
+F 2 "Resistor_SMD:R_1206_3216Metric" V 3430 3450 50  0001 C CNN
 F 3 "~" H 3500 3450 50  0001 C CNN
 	1    3500 3450
@@
 F 0 "R4" V 4193 3250 50  0000 C CNN
 F 1 "10K" V 4284 3250 50  0000 C CNN
-F 2 "" V 4330 3250 50  0001 C CNN
+F 2 "Resistor_SMD:R_1206_3216Metric" V 4330 3250 50  0001 C CNN
 F 3 "~" H 4400 3250 50  0001 C CNN
 	1    4400 3250
@@
 F 0 "R7" V 5093 2950 50  0000 C CNN
 F 1 "100K" V 5184 2950 50  0000 C CNN
-F 2 "" V 5230 2950 50  0001 C CNN
+F 2 "Resistor_SMD:R_1206_3216Metric" V 5230 2950 50  0001 C CNN
 F 3 "~" H 5300 2950 50  0001 C CNN
 	1    5300 2950
@@
 F 0 "R5" V 4193 3650 50  0000 C CNN
 F 1 "10K" V 4284 3650 50  0000 C CNN
-F 2 "" V 4330 3650 50  0001 C CNN
+F 2 "Resistor_SMD:R_1206_3216Metric" V 4330 3650 50  0001 C CNN
 F 3 "~" H 4400 3650 50  0001 C CNN
 	1    4400 3650
@@
 F 0 "R6" H 4730 3904 50  0000 R CNN
 F 1 "10K" H 4730 3995 50  0000 R CNN
-F 2 "" V 4730 3950 50  0001 C CNN
+F 2 "Resistor_SMD:R_1206_3216Metric" V 4730 3950 50  0001 C CNN
 F 3 "~" H 4800 3950 50  0001 C CNN
 	1    4800 3950
@@
 F 0 "R8" V 6843 3750 50  0000 C CNN
 F 1 "10K" V 6934 3750 50  0000 C CNN
-F 2 "" V 6980 3750 50  0001 C CNN
+F 2 "Resistor_SMD:R_1206_3216Metric" V 6980 3750 50  0001 C CNN
 F 3 "~" H 7050 3750 50  0001 C CNN
 	1    7050 3750
@@
 F 0 "R10" H 7520 2796 50  0000 L CNN
 F 1 "10K" H 7520 2705 50  0000 L CNN
-F 2 "" V 7380 2750 50  0001 C CNN
+F 2 "Resistor_SMD:R_1206_3216Metric" V 7380 2750 50  0001 C CNN
 F 3 "~" H 7450 2750 50  0001 C CNN
 	1    7450 2750
@@
 F 0 "R11" V 7643 3750 50  0000 C CNN
 F 1 "100K" V 7734 3750 50  0000 C CNN
-F 2 "" V 7780 3750 50  0001 C CNN
+F 2 "Resistor_SMD:R_1206_3216Metric" V 7780 3750 50  0001 C CNN
 F 3 "~" H 7850 3750 50  0001 C CNN
 	1    7850 3750
@@
 F 0 "R9" V 6893 3050 50  0000 C CNN
 F 1 "10K" V 6984 3050 50  0000 C CNN
-F 2 "" V 7030 3050 50  0001 C CNN
+F 2 "Resistor_SMD:R_1206_3216Metric" V 7030 3050 50  0001 C CNN
 F 3 "~" H 7100 3050 50  0001 C CNN
 	1    7100 3050
@@
 F 0 "R2" H 3320 5546 50  0000 L CNN
 F 1 "1K" H 3320 5455 50  0000 L CNN
-F 2 "" V 3180 5500 50  0001 C CNN
+F 2 "Resistor_SMD:R_1206_3216Metric" V 3180 5500 50  0001 C CNN
 F 3 "~" H 3250 5500 50  0001 C CNN
 	1    3250 5500
@@
 F 0 "U1" H 5350 3817 50  0000 C CNN
 F 1 "LM358" H 5350 3726 50  0000 C CNN
-F 2 "" H 5350 3450 50  0001 C CNN
+F 2 "Package_SO:SOP-8_3.9x4.9mm_P1.27mm" H 5350 3450 50  0001 C CNN
 F 3 "http://www.ti.com/lit/ds/symlink/lm2904-n.pdf" H 5350 3450 50  0001 C CNN
+F 4 "Texas Instruments" H 5350 3450 50  0001 C CNN "Manf"
+F 5 "LM358AMX" H 5350 3450 50  0001 C CNN "Manf#"
+F 6 "LM358, Dual Operational Amplifiers" H 5350 3450 50  0001 C CNN "Desc"
+F 7 "LM358AMXTR-ND" H 5350 3450 50  0001 C CNN "Digikey# "
 	1    5350 3450
 	1    0    0    1
@@
 F 0 "U1" H 7900 3517 50  0000 C CNN
 F 1 "LM358" H 7900 3426 50  0000 C CNN
-F 2 "" H 7900 3150 50  0001 C CNN
+F 2 "Package_SO:SOP-8_3.9x4.9mm_P1.27mm" H 7900 3150 50  0001 C CNN
 F 3 "http://www.ti.com/lit/ds/symlink/lm2904-n.pdf" H 7900 3150 50  0001 C CNN
 	2    7900 3150
@@
 F 0 "U1" H 5108 5596 50  0000 L CNN
 F 1 "LM358" H 5108 5505 50  0000 L CNN
-F 2 "" H 5150 5550 50  0001 C CNN
+F 2 "Package_SO:SOP-8_3.9x4.9mm_P1.27mm" H 5150 5550 50  0001 C CNN
 F 3 "http://www.ti.com/lit/ds/symlink/lm2904-n.pdf" H 5150 5550 50  0001 C CNN
 	3    5150 5550
@@
 F 0 "C1" V 3648 3250 50  0000 C CNN
 F 1 "1u" V 3739 3250 50  0000 C CNN
-F 2 "" H 3938 3100 50  0001 C CNN
+F 2 "Capacitor_SMD:C_0805_2012Metric" H 3938 3100 50  0001 C CNN
 F 3 "~" H 3900 3250 50  0001 C CNN
 	1    3900 3250
@@
 F 0 "C2" V 5048 2550 50  0000 C CNN
 F 1 "1n" V 5139 2550 50  0000 C CNN
-F 2 "" H 5338 2400 50  0001 C CNN
+F 2 "Capacitor_SMD:C_0805_2012Metric" H 5338 2400 50  0001 C CNN
 F 3 "~" H 5300 2550 50  0001 C CNN
 	1    5300 2550
@@
 F 0 "C4" V 6298 3750 50  0000 C CNN
 F 1 "1u" V 6389 3750 50  0000 C CNN
-F 2 "" H 6588 3600 50  0001 C CNN
+F 2 "Capacitor_SMD:C_0805_2012Metric" H 6588 3600 50  0001 C CNN
 F 3 "~" H 6550 3750 50  0001 C CNN
 	1    6550 3750
@@
 F 0 "C5" V 7598 4150 50  0000 C CNN
 F 1 "1n" V 7689 4150 50  0000 C CNN
-F 2 "" H 7888 4000 50  0001 C CNN
+F 2 "Capacitor_SMD:C_0805_2012Metric" H 7888 4000 50  0001 C CNN
 F 3 "~" H 7850 4150 50  0001 C CNN
 	1    7850 4150
@@
 F 0 "C3" H 5815 5596 50  0000 L CNN
 F 1 "1n" H 5815 5505 50  0000 L CNN
-F 2 "" H 5738 5400 50  0001 C CNN
+F 2 "Capacitor_SMD:C_0805_2012Metric" H 5738 5400 50  0001 C CNN
 F 3 "~" H 5700 5550 50  0001 C CNN
 	1    5700 5550
@@
 F 0 "D1" V 3289 5882 50  0000 R CNN
 F 1 "LED_ALT" V 3198 5882 50  0000 R CNN
-F 2 "" H 3250 6000 50  0001 C CNN
+F 2 "LED_SMD:LED_1206_3216Metric" H 3250 6000 50  0001 C CNN
 F 3 "~" H 3250 6000 50  0001 C CNN
 	1    3250 6000
@@
 P 6050 3750
 F 0 "RV1" H 5981 3796 50  0000 R CNN
-F 1 "R_POT" H 5981 3705 50  0000 R CNN
-F 2 "" H 6050 3750 50  0001 C CNN
-F 3 "~" H 6050 3750 50  0001 C CNN
+F 1 "100K" H 5981 3705 50  0000 R CNN
+F 2 "Resistor_SMD:R_1206_3216Metric" H 6050 3750 50  0001 C CNN
+F 3 "https://www.bourns.com/pdfs/3296.pdf" H 6050 3750 50  0001 C CNN
+F 4 "Bourns Inc." H 6050 3750 50  0001 C CNN "Manf"
+F 5 "3296W-1-104LF" H 6050 3750 50  0001 C CNN "Manf#"
+F 6 "TRIMMER 100K OHM 0.5W PC PIN TOP" H 6050 3750 50  0001 C CNN "Desc"
+F 7 "3296W-104LF-ND" H 6050 3750 50  0001 C CNN "Digikey# "
 	1    6050 3750
 	1    0    0    -1
@@
 F 0 "J1" H 1118 3175 50  0000 C CNN
 F 1 "Conn_01x02" H 1118 3266 50  0000 C CNN
-F 2 "" H 1200 3500 50  0001 C CNN
-F 3 "~" H 1200 3500 50  0001 C CNN
+F 2 "TerminalBlock_Phoenix:TerminalBlock_Phoenix_MKDS-1,5-2-5.08_1x02_P5.08mm_Horizontal" H 1200 3500 50  0001 C CNN
+F 3 "https://www.phoenixcontact.com/online/portal/pi/pxc/product_detail_page/!ut/p/z1/5VdNT-MwEP0r3UNvuHa-3WNId5e0bLfQAk0ukZ04lSFfJKYFfv3abVAFgnBAHFaJRortzIz9nmciPRjCNQwLsuUbInhZkEzOg9COsD7zzn6b2h907Xvowvi7unSm7ng6s-E1DGHYsIzFgiUeEWxT1k8wcM_P1QdBKAw0Nari-A4GC6BpAEmz1FrGaU2Ud8VZsXfiiXTHGNvYUfMyXXje7G2Y4CJjctE7HQhW51yec0CzMr4bgMGf2WQ5H-gn1hANdGCdICwXXzLedIExzmXybqyHePTB46LP4gMZ73zosNTgUsHjRSNIETPFxbssHUmtmXTbsvrgWNVl8hCLCROEZ40vWO6_pvPDa3rLe5WkeZmwNm3ZcFUNrzaR8xV7FO3aO3crU2Sk2DyQjUrzCXKjr8h11Fvkem-R97bP9d72ud_bPvd72-d-b_vc722fu72tdre3fzjXksgDDwbLZ306uYBTSQLNR7s4H6FR9RiP2k2jZA8tqlRSqav47f196MIwLguhDrNWDA3RjtEhygmXwzawGaKMN2IfKMdS90Qvuifa654mOp5-iOxxoukxSQBNKANmalFAqUaBbjvU0Q0Ts7GSMmGXWtmLob1Dh9pZsiKa_IwWa2_hd3N06pjwZsvZDl4VZZ1LXbk8MK9uLqVU121zDMaOhYBpjzHAtkWAw2LDoCzWYszgGfpsB_uLO3Snn5vfm9761vS_vnr6aVexnF6id-tZFvCxoss0bT8MEavrsj6UM6zyHButgav184rR59eGkXF0OVg0n1vbN_a_ReInA92awXS7263S3KO4fT3tfvwD5torBw!!/p0/IZ7_82KCHG41M0VIC0Q3OTR7JA9JI2=CZ6_82KCHG41M0VIC0Q3OTR7JA9JK6=LA0=EdownloadId!7570218=action!downloadFile==/#Z7_82KCHG41M0VIC0Q3OTR7JA9JI2" H 1200 3500 50  0001 C CNN
+F 4 "Phoenix Contact" H 1200 3500 50  0001 C CNN "Manf"
+F 5 "1888687" H 1200 3500 50  0001 C CNN "Manf#"
+F 6 "PCB terminal block - MKDSN 2,5/ 2-5,08" H 1200 3500 50  0001 C CNN "Desc"
+F 7 "277-5893-ND" H 1200 3500 50  0001 C CNN "Digikey#"
 	1    1200 3500
 	-1   0    0    1
@@
 F 0 "J2" H 9880 3242 50  0000 L CNN
 F 1 "Conn_01x04" H 9880 3151 50  0000 L CNN
-F 2 "" H 9800 3250 50  0001 C CNN
+F 2 "Connector_PinHeader_2.54mm:PinHeader_1x04_P2.54mm_Vertical" H 9800 3250 50  0001 C CNN
 F 3 "~" H 9800 3250 50  0001 C CNN
 	1    9800 3250
@@
 Text Notes 850  3850 0    50   ~ 0
 High Voltage AC Input
+Text Notes 6100 4000 0    50   ~ 0
+Gain Adjustment
 $EndSCHEMATC

Commit message: Se agrego/arreglo segun revision de Felipe
Parts:
- D1: Desc (none) -> Led Red SMD 1206
- T1: footprint ZMPT101B:XFMR_ZMPT101B -> tp:XFMR_ZMPT101B
Changed lines of the file:
@@
 F 0 "T1" H 2666 3840 50  0000 C CNN
 F 1 "ZMPT101B" H 2666 3749 50  0000 C CNN
-F 2 "ZMPT101B:XFMR_ZMPT101B" H 2600 3450 50  0001 L BNN
+F 2 "tp:XFMR_ZMPT101B" H 2600 3450 50  0001 L BNN
 F 3 "https://www.datasheet4u.com/datasheet-pdf/ZemingLangxi/ZMPT101B/pdf.php?id=1381510" H 2600 3450 50  0001 L BNN
 F 4 "Qingxian Zeming Langxi Electronic" H 2600 3450 50  0001 C CNN "Manf"
@@
 F 2 "LED_SMD:LED_1206_3216Metric" H 3250 6000 50  0001 C CNN
 F 3 "~" H 3250 6000 50  0001 C CNN
+F 4 "Led Red SMD 1206" V 3250 6000 50  0001 C CNN "Desc"
 	1    3250 6000
 	0    -1   -1   0

Commit message: Posicionamiento de componentes en PCB
Parts:
- RV1: footprint Resistor_SMD:R_1206_3216Metric -> Potentiometer_THT:Potentiometer_Bourns_3296W_Vertical
- U1: footprint Package_SO:SOP-8_3.9x4.9mm_P1.27mm -> Package_SO:SOIC-8_3.9x4.9mm_P1.27mm
Connections:
- net at T1.2: now also J1.2 (Pin_2); no longer J1.1 (Pin_1)
- net at R1.2: now also J1.1 (Pin_1); no longer J1.2 (Pin_2)
Changed lines of the file:
@@
-$EndComp
-$Comp
-L Device:R R1
-U 1 1 605552F6
-P 1900 3250
-F 0 "R1" V 1693 3250 50  0000 C CNN
-F 1 "820K" V 1784 3250 50  0000 C CNN
-F 2 "Resistor_SMD:R_1206_3216Metric" V 1830 3250 50  0001 C CNN
-F 3 "~" H 1900 3250 50  0001 C CNN
-	1    1900 3250
-	0    1    1    0
 $EndComp
 $Comp
@@
 F 0 "U1" H 5350 3817 50  0000 C CNN
 F 1 "LM358" H 5350 3726 50  0000 C CNN
-F 2 "Package_SO:SOP-8_3.9x4.9mm_P1.27mm" H 5350 3450 50  0001 C CNN
+F 2 "Package_SO:SOIC-8_3.9x4.9mm_P1.27mm" H 5350 3450 50  0001 C CNN
 F 3 "http://www.ti.com/lit/ds/symlink/lm2904-n.pdf" H 5350 3450 50  0001 C CNN
 F 4 "Texas Instruments" H 5350 3450 50  0001 C CNN "Manf"
@@
 F 0 "U1" H 7900 3517 50  0000 C CNN
 F 1 "LM358" H 7900 3426 50  0000 C CNN
-F 2 "Package_SO:SOP-8_3.9x4.9mm_P1.27mm" H 7900 3150 50  0001 C CNN
+F 2 "Package_SO:SOIC-8_3.9x4.9mm_P1.27mm" H 7900 3150 50  0001 C CNN
 F 3 "http://www.ti.com/lit/ds/symlink/lm2904-n.pdf" H 7900 3150 50  0001 C CNN
 	2    7900 3150
@@
 F 0 "U1" H 5108 5596 50  0000 L CNN
 F 1 "LM358" H 5108 5505 50  0000 L CNN
-F 2 "Package_SO:SOP-8_3.9x4.9mm_P1.27mm" H 5150 5550 50  0001 C CNN
+F 2 "Package_SO:SOIC-8_3.9x4.9mm_P1.27mm" H 5150 5550 50  0001 C CNN
 F 3 "http://www.ti.com/lit/ds/symlink/lm2904-n.pdf" H 5150 5550 50  0001 C CNN
 	3    5150 5550
@@
 F 0 "RV1" H 5981 3796 50  0000 R CNN
 F 1 "100K" H 5981 3705 50  0000 R CNN
-F 2 "Resistor_SMD:R_1206_3216Metric" H 6050 3750 50  0001 C CNN
+F 2 "Potentiometer_THT:Potentiometer_Bourns_3296W_Vertical" H 6050 3750 50  0001 C CNN
 F 3 "https://www.bourns.com/pdfs/3296.pdf" H 6050 3750 50  0001 C CNN
 F 4 "Bourns Inc." H 6050 3750 50  0001 C CNN "Manf"
@@
 L Connector_Generic:Conn_01x02 J1
 U 1 1 6056CAEF
-P 1200 3500
-F 0 "J1" H 1118 3175 50  0000 C CNN
-F 1 "Conn_01x02" H 1118 3266 50  0000 C CNN
-F 2 "TerminalBlock_Phoenix:TerminalBlock_Phoenix_MKDS-1,5-2-5.08_1x02_P5.08mm_Horizontal" H 1200 3500 50  0001 C CNN
-F 3 "https://www.phoenixcontact.com/online/portal/pi/pxc/product_detail_page/!ut/p/z1/5VdNT-MwEP0r3UNvuHa-3WNId5e0bLfQAk0ukZ04lSFfJKYFfv3abVAFgnBAHFaJRortzIz9nmciPRjCNQwLsuUbInhZkEzOg9COsD7zzn6b2h907Xvowvi7unSm7ng6s-E1DGHYsIzFgiUeEWxT1k8wcM_P1QdBKAw0Nari-A4GC6BpAEmz1FrGaU2Ud8VZsXfiiXTHGNvYUfMyXXje7G2Y4CJjctE7HQhW51yec0CzMr4bgMGf2WQ5H-gn1hANdGCdICwXXzLedIExzmXybqyHePTB46LP4gMZ73zosNTgUsHjRSNIETPFxbssHUmtmXTbsvrgWNVl8hCLCROEZ40vWO6_pvPDa3rLe5WkeZmwNm3ZcFUNrzaR8xV7FO3aO3crU2Sk2DyQjUrzCXKjr8h11Fvkem-R97bP9d72ud_bPvd72-d-b_vc722fu72tdre3fzjXksgDDwbLZ306uYBTSQLNR7s4H6FR9RiP2k2jZA8tqlRSqav47f196MIwLguhDrNWDA3RjtEhygmXwzawGaKMN2IfKMdS90Qvuifa654mOp5-iOxxoukxSQBNKANmalFAqUaBbjvU0Q0Ts7GSMmGXWtmLob1Dh9pZsiKa_IwWa2_hd3N06pjwZsvZDl4VZZ1LXbk8MK9uLqVU121zDMaOhYBpjzHAtkWAw2LDoCzWYszgGfpsB_uLO3Snn5vfm9761vS_vnr6aVexnF6id-tZFvCxoss0bT8MEavrsj6UM6zyHButgav184rR59eGkXF0OVg0n1vbN_a_ReInA92awXS7263S3KO4fT3tfvwD5torBw!!/p0/IZ7_82KCHG41M0VIC0Q3OTR7JA9JI2=CZ6_82KCHG41M0VIC0Q3OTR7JA9JK6=LA0=EdownloadId!7570218=action!downloadFile==/#Z7_82KCHG41M0VIC0Q3OTR7JA9JI2" H 1200 3500 50  0001 C CNN
-F 4 "Phoenix Contact" H 1200 3500 50  0001 C CNN "Manf"
-F 5 "1888687" H 1200 3500 50  0001 C CNN "Manf#"
-F 6 "PCB terminal block - MKDSN 2,5/ 2-5,08" H 1200 3500 50  0001 C CNN "Desc"
-F 7 "277-5893-ND" H 1200 3500 50  0001 C CNN "Digikey#"
-	1    1200 3500
-	-1   0    0    1
+P 1200 3400
+F 0 "J1" H 1118 3075 50  0000 C CNN
+F 1 "Conn_01x02" H 1118 3166 50  0000 C CNN
+F 2 "TerminalBlock_Phoenix:TerminalBlock_Phoenix_MKDS-1,5-2-5.08_1x02_P5.08mm_Horizontal" H 1200 3400 50  0001 C CNN
+F 3 "https://www.phoenixcontact.com/online/portal/pi/pxc/product_detail_page/!ut/p/z1/5VdNT-MwEP0r3UNvuHa-3WNId5e0bLfQAk0ukZ04lSFfJKYFfv3abVAFgnBAHFaJRortzIz9nmciPRjCNQwLsuUbInhZkEzOg9COsD7zzn6b2h907Xvowvi7unSm7ng6s-E1DGHYsIzFgiUeEWxT1k8wcM_P1QdBKAw0Nari-A4GC6BpAEmz1FrGaU2Ud8VZsXfiiXTHGNvYUfMyXXje7G2Y4CJjctE7HQhW51yec0CzMr4bgMGf2WQ5H-gn1hANdGCdICwXXzLedIExzmXybqyHePTB46LP4gMZ73zosNTgUsHjRSNIETPFxbssHUmtmXTbsvrgWNVl8hCLCROEZ40vWO6_pvPDa3rLe5WkeZmwNm3ZcFUNrzaR8xV7FO3aO3crU2Sk2DyQjUrzCXKjr8h11Fvkem-R97bP9d72ud_bPvd72-d-b_vc722fu72tdre3fzjXksgDDwbLZ306uYBTSQLNR7s4H6FR9RiP2k2jZA8tqlRSqav47f196MIwLguhDrNWDA3RjtEhygmXwzawGaKMN2IfKMdS90Qvuifa654mOp5-iOxxoukxSQBNKANmalFAqUaBbjvU0Q0Ts7GSMmGXWtmLob1Dh9pZsiKa_IwWa2_hd3N06pjwZsvZDl4VZZ1LXbk8MK9uLqVU121zDMaOhYBpjzHAtkWAw2LDoCzWYszgGfpsB_uLO3Snn5vfm9761vS_vnr6aVexnF6id-tZFvCxoss0bT8MEavrsj6UM6zyHButgav184rR59eGkXF0OVg0n1vbN_a_ReInA92awXS7263S3KO4fT3tfvwD5torBw!!/p0/IZ7_82KCHG41M0VIC0Q3OTR7JA9JI2=CZ6_82KCHG41M0VIC0Q3OTR7JA9JK6=LA0=EdownloadId!7570218=action!downloadFile==/#Z7_82KCHG41M0VIC0Q3OTR7JA9JI2" H 1200 3400 50  0001 C CNN
+F 4 "Phoenix Contact" H 1200 3400 50  0001 C CNN "Manf"
+F 5 "1888687" H 1200 3400 50  0001 C CNN "Manf#"
+F 6 "PCB terminal block - MKDSN 2,5/ 2-5,08" H 1200 3400 50  0001 C CNN "Desc"
+F 7 "277-5893-ND" H 1200 3400 50  0001 C CNN "Digikey#"
+	1    1200 3400
+	-1   0    0    -1
 $EndComp
 $Comp
@@
 Text Notes 6100 4000 0    50   ~ 0
 Gain Adjustment
+$Comp
+L Device:R R1
+U 1 1 605552F6
+P 1900 3250
+F 0 "R1" V 1693 3250 50  0000 C CNN
+F 1 "820K" V 1784 3250 50  0000 C CNN
+F 2 "Resistor_SMD:R_1206_3216Metric" V 1830 3250 50  0001 C CNN
+F 3 "~" H 1900 3250 50  0001 C CNN
+	1    1900 3250
+	0    1    1    0
+$EndComp
 $EndSCHEMATC

Commit message: Avance de PCB. Agregado de agujeros de fijacion
Parts:
- added FID1: Fiducial, Fiducial:Fiducial_0.5mm_Mask1.5mm, symbol Mechanical:Fiducial
- added H1, H2, H3, H4: MountingHole, MountingHole:MountingHole_2.1mm, symbol Mechanical:MountingHole
Changed lines of the file:
@@
 Wire Wire Line
 	5700 5700 5700 6050
-Text Label 8850 3150 0    50   ~ 0
+Text Label 8600 3150 0    50   ~ 0
 OUT
 Text Notes 850  3850 0    50   ~ 0
@@
 	0    1    1    0
 $EndComp
+$Comp
+L power:PWR_FLAG #FLG0101
+U 1 1 60747F6D
+P 9000 2900
+F 0 "#FLG0101" H 9000 2975 50  0001 C CNN
+F 1 "PWR_FLAG" H 9000 3073 50  0000 C CNN
+F 2 "" H 9000 2900 50  0001 C CNN
+F 3 "~" H 9000 2900 50  0001 C CNN
+	1    9000 2900
+	1    0    0    -1
+$EndComp
+$Comp
+L power:PWR_FLAG #FLG0102
+U 1 1 6074901F
+P 9000 3450
+F 0 "#FLG0102" H 9000 3525 50  0001 C CNN
+F 1 "PWR_FLAG" H 9000 3623 50  0000 C CNN
+F 2 "" H 9000 3450 50  0001 C CNN
+F 3 "~" H 9000 3450 50  0001 C CNN
+	1    9000 3450
+	-1   0    0    1
+$EndComp
+Wire Wire Line
+	9300 3350 9000 3350
+Wire Wire Line
+	9000 3350 9000 3450
+Wire Wire Line
+	9300 3050 9000 3050
+Wire Wire Line
+	9000 3050 9000 2900
+Connection ~ 9300 3050
+$Comp
+L Mechanical:MountingHole H1
+U 1 1 6074EA99
+P 1500 5200
+F 0 "H1" H 1600 5246 50  0000 L CNN
+F 1 "MountingHole" H 1600 5155 50  0000 L CNN
+F 2 "MountingHole:MountingHole_2.1mm" H 1500 5200 50  0001 C CNN
+F 3 "~" H 1500 5200 50  0001 C CNN
+	1    1500 5200
+	1    0    0    -1
+$EndComp
+$Comp
+L Mechanical:MountingHole H2
+U 1 1 6074F120
+P 1500 5550
+F 0 "H2" H 1600 5596 50  0000 L CNN
+F 1 "MountingHole" H 1600 5505 50  0000 L CNN
+F 2 "MountingHole:MountingHole_2.1mm" H 1500 5550 50  0001 C CNN
+F 3 "~" H 1500 5550 50  0001 C CNN
+	1    1500 5550
+	1    0    0    -1
+$EndComp
+$Comp
+L Mechanical:MountingHole H3
+U 1 1 6074F65C
+P 1500 5900
+F 0 "H3" H 1600 5946 50  0000 L CNN
+F 1 "MountingHole" H 1600 5855 50  0000 L CNN
+F 2 "MountingHole:MountingHole_2.1mm" H 1500 5900 50  0001 C CNN
+F 3 "~" H 1500 5900 50  0001 C CNN
+	1    1500 5900
+	1    0    0    -1
+$EndComp
+$Comp
+L Mechanical:MountingHole H4
+U 1 1 6074FC40
+P 1500 6250
+F 0 "H4" H 1600 6296 50  0000 L CNN
+F 1 "MountingHole" H 1600 6205 50  0000 L CNN
+F 2 "MountingHole:MountingHole_2.1mm" H 1500 6250 50  0001 C CNN
+F 3 "~" H 1500 6250 50  0001 C CNN
+	1    1500 6250
+	1    0    0    -1
+$EndComp
+$Comp
+L Mechanical:Fiducial FID1
+U 1 1 607503FD
+P 1500 6600
+F 0 "FID1" H 1585 6646 50  0000 L CNN
+F 1 "Fiducial" H 1585 6555 50  0000 L CNN
+F 2 "Fiducial:Fiducial_0.5mm_Mask1.5mm" H 1500 6600 50  0001 C CNN
+F 3 "~" H 1500 6600 50  0001 C CNN
+	1    1500 6600
+	1    0    0    -1
+$EndComp
 $EndSCHEMATC

Commit message: Se aplicaron todos los comentarios hechos en la revisión del docente
Parts:
- C1, C4: value 1u -> 1uF
- C2, C3, C5: value 1n -> 1nF
- D1: value LED_ALT -> SMD Red Led; Desc Led Red SMD 1206 -> LED RED CLEAR 1206 SMD; Digikey#  (none) -> 1830-1092-2-ND; Manf (none) -> Inolux; Manf# (none) -> IN-S126ATR
- R1, R10, R11, R2, R3, R4, R5, R6, R7, R8, R9: footprint Resistor_SMD:R_1206_3216Metric -> Resistor_SMD:R_0805_2012Metric
- U1: Desc (none) -> LM358, Dual Operational Amplifiers; Digikey#  (none) -> LM358AMXTR-ND; Manf (none) -> Texas Instruments; Manf# (none) -> LM358AMX
Other:
- note added: "First OP stage - Pre-Amplifier"
- note added: "Second OP stage - Output stage"
- moved on the sheet: C4, C5, J1, J2, R1, R10, R11, R8, R9, RV1, T1, U1B

Commit message: Proyecto actualizado según revisión  F. Calcavecchia 18/04/2021
Parts:
- added FID2: Fiducial, Fiducial:Fiducial_0.5mm_Mask1.5mm, symbol Mechanical:Fiducial
Changed lines of the file:
@@
 	2750 3650 3500 3650
 Connection ~ 3500 3650
+$Comp
+L Mechanical:Fiducial FID2
+U 1 1 607DD604
+P 1500 6850
+F 0 "FID2" H 1585 6896 50  0000 L CNN
+F 1 "Fiducial" H 1585 6805 50  0000 L CNN
+F 2 "Fiducial:Fiducial_0.5mm_Mask1.5mm" H 1500 6850 50  0001 C CNN
+F 3 "~" H 1500 6850 50  0001 C CNN
+	1    1500 6850
+	1    0    0    -1
+$EndComp
 $EndSCHEMATC
